File: pcb/lul.sch (EAGLE design)
At the start: 85 parts, among them IC1 STM32F072C8T6, IC2 REG1117, IC3 74AHCT1G08DBV, SW1 324_SW324_SWITCH_FOOT_HOLE, SW2 324_SW324_SWITCH_FOOT_HOLE, SW3 324_SW324_SWITCH_FOOT_HOLE, SW4 324_SW324_SWITCH_FOOT_HOLE, U1 UG-2864HSWEG01, U2 USBC_16P

Commit message: simpler version for jlcpcb assembly
Parts:
- removed C28, C3, C4, C6: 1uF, clock:CAP0805
- removed C5, C7, C8: 2.2uF, clock:CAP0805
- removed R17: 10K, clock:RESISTOR0805-RES
- removed R3: 560K, clock:RESISTOR0805-RES
- removed R7, R8: 5.1K, clock:RESISTOR0805-RES
- removed U1: UG-2864HSWEG01, lul:LUL_DISP_OLED_UG-2864HSWEG01
- added U$2: OLED_0.96_I2C, tft_1.8_1.44_oled_0.96:OLED_0.96_I2C
- LED1, LED10, LED11, LED12, LED13, LED14, LED15, LED2, LED3, LED4, LED5, LED6, LED7, LED8, LED9: value WS2812B3535 -> WS2812B-MINI; device lul:WS2812B3535 -> LED:WS2812B-MINI
Connections:
- removed net N$11: C28.2, C5.2, U1.VCC
- removed net N$12: C8.2, U1.VCOMH
- removed net N$3: R3.2, U1.IREF
- removed net N$4: C3.2, U1.C2P
- removed net N$5: C3.1, U1.C2N
- removed net N$6: C4.2, U1.C1P
- removed net N$7: C4.1, U1.C1N
- net +3V3: now also U$2.VCC; no longer C6.2, C7.2, R7.2, R8.2, U1.BS1, U1.VBAT, U1.VDD
- net GND: now also U$2.GND; no longer C28.1, C5.1, C6.1, C7.1, C8.1, R17.1, R3.1, U1./CS, U1.BS0, U1.BS2, U1.D3, U1.D4, U1.D5, U1.D6, U1.D7, U1.DC/I2C_SA0, U1.E/RD, U1.NC, U1.NC(GND)@1, U1.NC(GND)@2, U1.R/W, U1.VLSS, U1.VSS
- net N$15: now also LED1.DIN, LED2.DOUT; no longer LED1.DI, LED2.DO
- net N$17: now also LED1.DOUT, LED4.DIN; no longer LED1.DO, LED4.DI
- net N$18: now also LED4.DOUT, LED5.DIN; no longer LED4.DO, LED5.DI
- net N$19: now also LED5.DOUT, LED6.DIN; no longer LED5.DO, LED6.DI
- net N$20: now also LED6.DOUT, LED9.DIN; no longer LED6.DO, LED9.DI
- net N$21: now also LED8.DIN, LED9.DOUT; no longer LED8.DI, LED9.DO
- net N$22: now also LED7.DIN, LED8.DOUT; no longer LED7.DI, LED8.DO
- net N$23: now also LED10.DIN, LED7.DOUT; no longer LED10.DI, LED7.DO
- net N$24: now also LED10.DOUT, LED11.DIN; no longer LED10.DO, LED11.DI
- net N$25: now also LED11.DOUT, LED12.DIN; no longer LED11.DO, LED12.DI
- net N$26: now also LED12.DOUT, LED15.DIN; no longer LED12.DO, LED15.DI
- net N$27: now also LED14.DIN, LED15.DOUT; no longer LED14.DI, LED15.DO
- net N$28: now also LED13.DIN, LED14.DOUT; no longer LED13.DI, LED14.DO
- net N$29: now also LED3.DIN; no longer LED3.DI
- net N$9: now also LED2.DIN, LED3.DOUT; no longer LED2.DI, LED3.DO
- net OLED_RESET: no longer R17.2, U1./RES
- net SCL: now also U$2.SCL; no longer R7.1, U1.D0/SPI_SCLK/I2C_SCK
- net SDA: now also U$2.SDA; no longer R8.1, U1.D1/SPI_SDIN/I2C_SDA, U1.D2/I2C_SDA
